File: OXCLPC.brd (EAGLE design)
At the start: 49.5 x 18 mm, 5 parts

Commit message: updated and added gerbers
Parts:
- removed U$2: (no value), adapter8784:OXC
- added U$3: (no value), OXC_Library:OXC-005
Changed lines of the file:
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@@
 </element>
 <element name="U$1" library="adapter8784" package="TEST" value="" x="4.771" y="-22.297" smashed="yes" rot="MR0"/>
-<element name="U$2" library="adapter8784" package="OXC" value="" x="1.471" y="-18.894" smashed="yes"/>
+<element name="U$3" library="OXC_Library" package="OXC-005" value="" x="1.778" y="-18.288" smashed="yes"/>
 </elements>
 <signals>
